Commit message: Odo error left, but works

File: description/robot_core.xacro (robot description, xacro)
@@ -89,5 +89,5 @@
         <child link="right_wheel"/>
         <origin xyz="0 ${-wheel_offset_y} 0" rpy="${pi/2} 0 0" />
-        <axis xyz="0 0 -1"/>
+        <axis xyz="0 0 1"/>
     </joint>
     <link name="right_wheel">

File: description/ros2_control.xacro (robot description, xacro)
@@ -11,5 +11,5 @@
                 <param name="baud_rate">57600</param>
                 <param name="timeout">1000</param>
-                <param name="enc_counts_per_rev">3436</param>
+                <param name="enc_counts_per_rev">46</param>
             </hardware>
             <joint name="left_wheel_joint">

Commit message: Created core URDF

File: description/robot_core.xacro (robot description, xacro)
@@ -27,4 +27,7 @@
     <material name="red">
         <color rgba="1 0 0 1"/>
+    </material>
+    <material name="green">
+        <color rgba="0 1 0 0.8"/>
     </material>
     <!-- BASE LINK -->
